File: smart-tps.brd (EAGLE design)
At the start: 210.8 x 163.8 mm, 81 parts, among them U3 BQ27441-G1, U4 BQ24075

Commit message: Update schematic
Parts:
- removed C14: 2.2uF, SparkFun-Passives:0805
- removed C15, C16: 1uF X5R, SparkFun-Passives:0805
- removed C17, C19: 1uF, SparkFun-Passives:0603-CAP
- removed C18: 4.7uF/16V, SparkFun-Passives:1206
- removed FID5, FID6: FIDUCIAL1X2, SparkFun-Aesthetics:FIDUCIAL-1X2
- removed LOGO10, LOGO12: SFE_LOGO_FLAME.1_INCH, SparkFun-Aesthetics:SFE_LOGO_FLAME_.1
- removed LOGO11, LOGO5: OSHW-LOGOS, SparkFun-Aesthetics:OSHW-LOGO-S
- removed LOGO4: SFE_LOGO_NAME.1_INCH, SparkFun-Aesthetics:SFE_LOGO_NAME_.1
- removed LOGO6: SFE_LOGO_NAME_FLAME.1_INCH, SparkFun-Aesthetics:SFE_LOGO_NAME_FLAME_.1
- removed OLED2: OLED0.66, microView-temp:OLED-0.66-64X48
- removed R4: 390k, SparkFun-Passives:0603-RES
- removed R5: 10k, SparkFun-Passives:0603-RES
- removed SJ11: (no value), SparkFun-Passives:PAD-JUMPER-2-NC_BY_TRACE_NO_SILK
- removed SJ12: (no value), SparkFun-Passives:PAD-JUMPER-2-NO_YES_SILK
- removed SJ13: BS1, SparkFun-Passives:PAD-JUMPER-3-2OF3_NC_BY_PASTE_YES_SILK_FULL_BOX
- removed SJ14: BS2, SparkFun-Passives:PAD-JUMPER-3-2OF3_NC_BY_PASTE_YES_SILK_FULL_BOX
- removed SJ15: (no value), SparkFun-Passives:PAD-JUMPER-3-NO-TIGHT
- removed TP5, TP6: TEST-POINT3X5, SparkFun-Passives:PAD.03X.05
- added J2, J4: TERMBLOCK_1X2-3.5MM, microbuilder:1X2-3.5MM
- added J5, J6, J7, J8: SJ-63062A, SJ-63062A:CUI_SJ-63062A
- added JP2, JP4: (no value), microbuilder:1X06_ROUND_70
- added U$18, U$19, U$20, U$21, U$40, U$41, U$42, U$43: MOUNTINGHOLE2.5, microbuilder:MOUNTINGHOLE_2.5_PLATED
- moved FID3 93.2 mm to (31.4, 129.8)
- moved JP23 93.2 mm to (40.6, 128.3)
- moved STANDOFF5 93.2 mm to (33.0, 132.1)
- moved STANDOFF6 93.2 mm to (61.0, 132.1)
- moved C10 93.2 mm to (49.5, 120.0)
- moved C6 93.2 mm to (48.9, 116.8)
- moved C7 93.2 mm to (47.2, 115.6)
- moved C8 93.2 mm to (57.1, 121.0)
- moved C9 93.2 mm to (53.3, 125.7)
- moved D3 93.2 mm to (44.5, 132.7)
- moved D4 93.2 mm to (47.0, 132.7)
- moved FID4 93.2 mm to (59.7, 106.7)
- moved JP14 93.2 mm to (53.3, 132.5)
- moved JP15 93.2 mm to (36.2, 121.9)
- moved JP16 93.2 mm to (38.1, 102.9)
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Connections:
- removed net BS1: OLED2.9, SJ13.2
- removed net BS2: OLED2.10, SJ14.2
- removed net C1N1: C15.2, OLED2.5
- removed net C1P1: C15.1, OLED2.4
- removed net C2N1: C16.2, OLED2.3
- removed net C2P1: C16.1, OLED2.2
- removed net D0/SCK: JP6.4, OLED2.16
- removed net D1/MOSI: JP6.3, OLED2.17, SJ12.1
- removed net D2: JP6.5, OLED2.18, SJ12.2
- removed net IREF1: OLED2.24, R4.2
- removed net VCC: C14.1, OLED2.26, TP5.P$1, TP6.P$1
- removed net VCOMH1: C18.1, OLED2.25
- removed net VDD: C17.1, JP6.2, OLED2.8, R5.2, SJ11.2
- removed net VDD_PU1: R5.1, SJ13.1, SJ14.1, SJ15.1
- new net 3V3: ARDUINO_NANO1.2, JP2.1, JP4.1, JP6.2
- new net LGND: J5.2, J7.2
- new net LV+: J2.2, J5.1, JP2.6
- new net LV-: J2.1, J7.1, JP2.5
- new net MISO: ARDUINO_NANO1.30, JP6.5
- new net MOSI: ARDUINO_NANO1.29, JP6.3
- new net SCK: ARDUINO_NANO1.1, JP6.4
- new net SGND: J6.2, J8.2
- new net SV+: J4.2, J6.1, JP4.6
- new net SV-: J4.1, J8.1, JP4.5
- net CS: now also ARDUINO_NANO1.28; no longer OLED2.11
- net D/C: now also ARDUINO_NANO1.26; no longer OLED2.13, SJ15.2
- net D3: no longer OLED2.19
- net D4: no longer OLED2.20
- net D5: no longer OLED2.21
- net D6: no longer OLED2.22
- net D7: no longer OLED2.23
- net GND: now also JP2.2, JP4.2; no longer C14.2, C17.2, C18.2, C19.2, OLED2.1, OLED2.27, OLED2.28, OLED2.7, R4.1, SJ13.3, SJ14.3, SJ15.3
- net RD/E: no longer OLED2.15
- net RESET: now also ARDUINO_NANO1.27; no longer OLED2.12
- net SCL: now also ARDUINO_NANO1.9, JP2.3, JP4.3
- net SDA: now also ARDUINO_NANO1.8, JP2.4, JP4.4
- net VBAT: no longer C19.1, OLED2.6, SJ11.1
- net WR/RW: no longer OLED2.14
Routing:
- net 3V3: track 0.00 -> 121.3 mm
- net SCK: track 0.00 -> 60.7 mm
- net MISO: track 0.00 -> 56.2 mm
- net LV-: track 0.00 -> 56.0 mm
- net MOSI: track 0.00 -> 55.7 mm
- net SV+: track 0.00 -> 51.4 mm
- net SDA: track 17.7 -> 59.0 mm
- net SCL: track 17.8 -> 59.1 mm
- net LV+: track 0.00 -> 32.7 mm
- net VDD: track 27.9 -> 0.00 mm, vias 2 -> 0
- net RESET: track 14.4 -> 41.3 mm
- net D/C: track 18.1 -> 42.3 mm, vias 1 -> 0
- net CS: track 15.2 -> 39.2 mm
- net D1/MOSI: track 15.8 -> 0.00 mm, vias 1 -> 0
- net VDD_PU1: track 14.2 -> 0.00 mm
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- removed copper zone on layer 1, net BATTERY_IN
- removed copper zone on layer 1, net GND
Other:
- board size 210.8 x 163.8 mm -> 69.8 x 81.3 mm
- board text added: "Gnd"
- board text added: "INA219 DC"
- board text added: "Scl"
- board text added: "Sda"
- board text added: "Vcc"
- board text added: "Vin+"
- board text added: "Vin-"
- board text removed: "0"
- board text removed: "3V3"
- board text removed: "BS1"
- board text removed: "BS2"
- board text removed: "VD/VB"
- board text removed: "v04"

Commit message: Commit final version of PCB
Parts:
- removed C10, C8: 10uF, SparkFun-Capacitors:0805-CAP
- removed C6: 1.0uF, SparkFun-Capacitors:0603-CAP
- removed C7: 0.47uF, SparkFun-Capacitors:0603-CAP
- removed C9: 1.0uF, SparkFun-Capacitors:1206-CAP
- removed D3: BLUE, SparkFun-LED:LED-0603
- removed D4: RED, SparkFun-LED:LED-0603
- removed FID3, FID4: FIDUCIAL1X2, SparkFun-Aesthetics:FIDUCIAL-1X2
- removed JP14: (no value), SparkFun-Connectors:USB-AB-MICRO-SMD_V03
- removed JP15: (no value), SparkFun-Connectors:JST-2-SMD
- removed JP19, JP20: (no value), SparkFun-Connectors:SCREWTERMINAL-3.5MM-2-NS@1
- removed JP22: (no value), SparkFun-Connectors:JST-2-PTH-NS@1
- removed JP23, JP26: (no value), SparkFun-Connectors:1X02_NO_SILK@1
- removed JP25: (no value), SparkFun-Connectors:1X01_NO_SILK
- removed R18: 0.01, SparkFun-Resistors:1206
- removed R19, R20: 4.7K, SparkFun-Resistors:0603-RES
- removed R21: 590, SparkFun-Passives:0603-RES
- removed R22: 1.1k, SparkFun-Passives:0603-RES
- removed R23: 180, SparkFun-Resistors:0603-RES
- removed R24: 1K, SparkFun-Resistors:0603-RES
- removed R25, R32: 100k, SparkFun-Resistors:0603-RES
- removed R26, R27, R30, R34: 10K, SparkFun-Resistors:0603-RES
- removed R28: ILIM, SparkFun-Resistors:1/6W-RES
- removed R29: ISET, SparkFun-Resistors:1/6W-RES
- removed R31: TMR, SparkFun-Resistors:1/6W-RES
- removed R33: TS, SparkFun-Resistors:1/6W-RES
- removed S3: (no value), SparkFun-Electromechanical:SWITCH-SPST-SMD-A
- removed S4: (no value), SparkFun-Electromechanical:DIPSWITCH-02-50MIL
- removed SJ10: (no value), SparkFun-Passives:PAD-JUMPER-3-2OF3_NC_BY_TRACE_YES_SILK_FULL_BOX
- removed SJ6, SJ7, SJ8, SJ9: JUMPER-PAD-2-NC_BY_TRACE, SparkFun-Passives:PAD-JUMPER-2-NC_BY_TRACE_YES_SILK
- removed TP3, TP4: (no value), SparkFun-Passives:PAD.03X.04
- removed U3: BQ27441-G1, battery-management-temp:PDSO-N12
- removed U4: BQ24075, battery-management-temp:PVQFN-N16
- added J1: (no value), SparkFun-Connectors:2X4
- added S1: (no value), switch-omron:B3F-10XX
- added U1: MAX16054AZT+, MAX16054AZT:21-0114C_MXM
- moved STANDOFF5 116.9 mm to (67.3, 20.3), flipped to the bottom, turned to 90 degrees
- moved JP18 104.4 mm to (55.9, 19.1), flipped to the bottom, turned to 180 degrees
- moved STANDOFF6 84.1 mm to (67.3, 48.3), flipped to the bottom, turned to 90 degrees
- moved STANDOFF7 84.1 mm to (39.4, 20.3), flipped to the bottom, turned to 90 degrees
- moved JP17 80.1 mm to (59.7, 44.5), flipped to the bottom, turned to 90 degrees
- moved JP16 77.5 mm to (38.1, 25.4), flipped to the bottom, turned to 90 degrees
- moved U$42 68.0 mm to (3.43, 69.2), turned to 0 degrees
- moved JP24 66.0 mm to (38.1, 38.1), flipped to the bottom, turned to 270 degrees
- moved JP21 62.3 mm to (38.1, 43.2), flipped to the bottom, turned to 270 degrees
- moved U$41 60.1 mm to (3.43, 52.1), turned to 0 degrees
- moved STANDOFF8 59.9 mm to (39.4, 48.3), flipped to the bottom, turned to 90 degrees
- moved J6 53.3 mm to (15.2, 80.0)
- moved J8 53.3 mm to (54.6, 80.0)
- moved J4 49.8 mm to (13.7, 68.4), turned to 180 degrees
- moved JP6 43.0 mm to (45.3, 39.1), turned to 270 degrees
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Connections:
- removed net !CHG!1: R23.2, U4.9
- removed net !PGOOD!1: SJ10.1, U4.7
- removed net 1.8V: C7.1, JP25.1, U3.5
- removed net D+: JP14.D+1, TP4.P$1
- removed net D-: JP14.D-1, TP3.P$1
- removed net EN1: R26.2, S4.4, U4.6
- removed net EN2: R27.2, S4.3, U4.5
- removed net ILIM1: R28.2, SJ7.2, U4.12
- removed net ISET1: R29.2, SJ8.2, U4.16
- removed net N$10: R22.1, SJ7.1
- removed net N$13: R21.1, SJ8.1
- removed net N$14: R24.2, SJ10.2
- removed net N$6: D3.C, R23.1
- removed net N$7: D4.C, R24.1
- removed net N$8: R32.2, S3.1
- removed net N$9: R30.1, SJ6.2
- removed net OUT: C8.1, D3.A, D4.A, JP20.1, JP21.2, JP22.2, R26.1, R27.1, U4.10, U4.11
- removed net SHIELD: JP14.SHIELD1, JP14.SHIELD2, JP14.SHIELD3
- removed net TMR1: R31.2, SJ9.2, U4.14
- removed net TS: R30.2, R33.2, U3.10, U4.1
- removed net USB_ID: JP14.ID1
- removed net V_BATT: C10.1, R18.1, R32.1, U3.7, U4.2, U4.3
- removed net V_USB: C9.1, JP14.VBUS1, JP19.1, JP23.1, JP26.1, U4.13
- new net AOFF: ARDUINO_NANO1.25, U1.3
- new net LTB: ARDUINO_NANO1.20, J1.2
- new net LTL: ARDUINO_NANO1.21, J1.4
- new net LTS: ARDUINO_NANO1.22, J1.6
- new net N$4: S1.1, U1.1
- new net TLV+: J1.5, JP2.6
- new net TLV-: J1.7, JP2.5
- new net TSV+: J1.1, JP4.6
- new net TSV-: J1.3, JP4.5
- net !CE!: no longer R25.1, U4.4
- net 3V3: now also JP21.2
- net BATTERY_IN: now also U1.6; no longer C6.1, JP15.2, R18.2, U3.6, U3.8
- net GND: now also J1.8, S1.3, U1.2; no longer C10.2, C6.2, C7.2, C8.2, C9.2, JP14.GND1, JP15.1, JP19.2, JP20.2, JP22.1, JP23.2, JP26.2, R21.2, R22.2, R25.2, R28.1, R29.1, R31.1, R33.1, S3.3, S4.1, S4.2, SJ10.3, SJ6.1, SJ9.1, U3.3, U3.EP, U3.EP1, U3.EP2, U3.EP3, U3.EP4, U4.8, U4.EP
- net GPOUT: no longer R34.1, U3.12
- net LV+: no longer JP2.6
- net LV-: no longer JP2.5
- net SCL: no longer R20.1, U3.2
- net SDA: no longer R19.1, U3.1
- net SV+: no longer JP4.6
- net SV-: no longer JP4.5
- net SYSOFF: now also U1.4; no longer S3.2, U4.15
- net V_PU: no longer R19.2, R20.2, R34.2
Routing:
- net OUT: track 56.2 -> 0.00 mm, vias 4 -> 0
- net SV+: track 51.4 -> 11.6 mm
- net TMR1: track 38.0 -> 0.00 mm, vias 3 -> 0
- net SV-: track 13.5 -> 48.3 mm
- net GPOUT: track 32.0 -> 0.00 mm, vias 1 -> 0
- net TS: track 30.3 -> 0.00 mm, vias 3 -> 0
- net MOSI: track 55.7 -> 28.1 mm
- net SDA: track 59.0 -> 86.1 mm, vias 0 -> 1
- net V_USB: track 27.0 -> 0.00 mm, vias 1 -> 0
- net TLV+: track 0.00 -> 25.8 mm, vias 0 -> 1
- net !CE!: track 24.9 -> 0.00 mm, vias 1 -> 0
- net SCL: track 59.1 -> 81.9 mm
- net !CHG!1: track 22.4 -> 0.00 mm, vias 2 -> 0
- net ISET1: track 22.1 -> 0.00 mm, vias 1 -> 0
- net TLV-: track 0.00 -> 21.8 mm, vias 0 -> 1
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- added copper zone on layer 1, net GND
- removed copper zone on layer 1, net OUT
- removed copper zone on layer 1, net SHIELD
- removed copper zone on layer 16, net SHIELD
- removed copper zone on layer 1, net V_BATT
- removed copper zone on layer 1, net V_USB
Other:
- board size 69.8 x 81.3 mm -> 69.8 x 88.9 mm
- board text added: "LTB"
- board text added: "LTL"
- board text added: "LTS"
- board text added: "ON/OFF"
- board text added: "TLV+"
- board text added: "TLV-"
- board text added: "TSV+"
- board text added: "TSV-"
- board text added: "UPD"
- board text added: "smart-tps v1.0 2020-11-03 Design by @vincetavernier"
- board text removed: "!CE!"
- board text removed: "!PGD!"
- board text removed: "1"
- board text removed: "1.8V"
- board text removed: "100mA"
- board text removed: "1s LiPo"
- board text removed: "2"
- board text removed: "3.3-4.2V"
- board text removed: "4.35-6.4V"
- board text removed: "500mA"
- board text removed: "BATT"
- board text removed: "Battery Babysitter"
- board text removed: "CHG"
- board text removed: "Charge"
- board text removed: "D+"
- board text removed: "D-"
- board text removed: "EN"
- board text removed: "EN1"
- board text removed: "EN2"
- board text removed: "GPOUT"
- board text removed: "I"
- board text removed: "ILIM"
- board text removed: "IN"
- board text removed: "ISET"
- board text removed: "OFF"
- board text removed: "ON"
- board text removed: "OUT"
- board text removed: "PWR-LED SEL"
- board text removed: "SCL"
- board text removed: "SDA"
- board text removed: "SYSOFF"
- board text removed: "TMR"
- board text removed: "TMR Set"
- board text removed: "TS"
- board text removed: "TS Disable"
- board text removed: "V"
- board text removed: "VPU"
- board text removed: "v10"
