File: smart-tps.sch (EAGLE design)
At the start: 80 parts, among them U3 BQ27441-G1, U4 BQ24075

Commit message: Update schematic
Parts:
- removed C14: 2.2uF, SparkFun-Passives:CAP0805
- removed C15, C16: 1uF X5R, SparkFun-Passives:CAP0805
- removed C17, C19: 1uF, SparkFun-Passives:CAP0603-CAP
- removed C18: 4.7uF/16V, SparkFun-Passives:CAP1206
- removed FID5, FID6: FIDUCIAL1X2, SparkFun-Aesthetics:FIDUCIAL1X2
- removed LOGO10: SFE_LOGO_FLAME.1_INCH, SparkFun-Aesthetics:SFE_LOGO_FLAME.1_INCH
- removed LOGO11, LOGO5: OSHW-LOGOS, SparkFun-Aesthetics:OSHW-LOGOS
- removed LOGO4: SFE_LOGO_NAME.1_INCH, SparkFun-Aesthetics:SFE_LOGO_NAME.1_INCH
- removed LOGO6: SFE_LOGO_NAME_FLAME.1_INCH, SparkFun-Aesthetics:SFE_LOGO_NAME_FLAME.1_INCH
- removed OLED2: OLED0.66, microView-temp:OLED0.66
- removed R4: 390k, SparkFun-Passives:RESISTOR0603-RES
- removed R5: 10k, SparkFun-Passives:RESISTOR0603-RES
- removed SJ11: JUMPER-PAD-2-NC_BY_TRACENO_SILK, SparkFun-Passives:JUMPER-PAD-2-NC_BY_TRACENO_SILK
- removed SJ12: JUMPER-PAD-2-NOYES_SILK, SparkFun-Passives:JUMPER-PAD-2-NOYES_SILK
- removed SJ13: BS1, SparkFun-Passives:JUMPER-PAD-3-2OF3_NC_BY_PASTE
- removed SJ14: BS2, SparkFun-Passives:JUMPER-PAD-3-2OF3_NC_BY_PASTE
- removed SJ15: JUMPER-PAD-3-NOTIGHT, SparkFun-Passives:JUMPER-PAD-3-NOTIGHT
- removed TP5, TP6: TEST-POINT3X5, SparkFun-Passives:TEST-POINT3X5
- added J2, J4: TERMBLOCK_1X2-3.5MM, microbuilder:TERMBLOCK_1X2-3.5MM
- added J5, J6, J7, J8: SJ-63062A, SJ-63062A:SJ-63062A
- added JP2, JP4: (no value), microbuilder:HEADER-1X670MIL
- added U$18, U$19, U$20, U$21, U$40, U$41, U$42, U$43: MOUNTINGHOLE2.5, microbuilder:MOUNTINGHOLE2.5
Connections:
- removed net BS1: OLED2.BS1, SJ13.2
- removed net BS2: OLED2.BS2, SJ14.2
- removed net C1N1: C15.2, OLED2.C1N
- removed net C1P1: C15.1, OLED2.C1P
- removed net C2N1: C16.2, OLED2.C2N
- removed net C2P1: C16.1, OLED2.C2P
- removed net D0/SCK: JP6.4, OLED2.D0/SCK
- removed net D1/MOSI: JP6.3, OLED2.D1/MOSI, SJ12.1
- removed net D2: JP6.5, OLED2.D2, SJ12.2
- removed net IREF1: OLED2.IREF, R4.2
- removed net VCC: C14.1, OLED2.VCC, TP5.1, TP6.1
- removed net VCOMH1: C18.1, OLED2.VCOMH
- removed net VDD: C17.1, JP6.2, OLED2.VDD, R5.2, SJ11.2
- removed net VDD_PU1: R5.1, SJ13.1, SJ14.1, SJ15.1
- new net 3V3: ARDUINO_NANO1.3V3, JP2.1, JP4.1, JP6.2
- new net LGND: J5.TIP, J7.TIP
- new net LV+: J2.2, J5.SLEEVE, JP2.6
- new net LV-: J2.1, J7.SLEEVE, JP2.5
- new net MISO: ARDUINO_NANO1.D12, JP6.5
- new net MOSI: ARDUINO_NANO1.D11, JP6.3
- new net SCK: ARDUINO_NANO1.D13, JP6.4
- new net SGND: J6.TIP, J8.TIP
- new net SV+: J4.2, J6.SLEEVE, JP4.6
- new net SV-: J4.1, J8.SLEEVE, JP4.5
- net CS: now also ARDUINO_NANO1.D10; no longer OLED2.!CS!
- net D/C: now also ARDUINO_NANO1.D8; no longer OLED2.D/!C!, SJ15.2
- net D3: no longer OLED2.D3
- net D4: no longer OLED2.D4
- net D5: no longer OLED2.D5
- net D6: no longer OLED2.D6
- net D7: no longer OLED2.D7
- net GND: now also JP2.2, JP4.2; no longer C14.2, C17.2, C18.2, C19.2, OLED2.GND@1, OLED2.GND@2, OLED2.VLSS, OLED2.VSS, R4.1, SJ13.3, SJ14.3, SJ15.3
- net RD/E: no longer OLED2.E/!RD!
- net RESET: now also ARDUINO_NANO1.D9; no longer OLED2.!RESET!
- net SCL: now also ARDUINO_NANO1.A5, JP2.3, JP4.3
- net SDA: now also ARDUINO_NANO1.A4, JP2.4, JP4.4
- net VBAT: no longer C19.1, OLED2.VBAT, SJ11.1
- net WR/RW: no longer OLED2.R/!W!
Other:
- note added: "OLED Connectors"
- note removed: "1.65 <= VDD <= 3.3"
- note removed: "3.3 <= VBAT <= 4.2"
- note removed: "In I2C mode, D/C sets the lower bit of the 7-bit address. Short it one way or the other. D/C I2C Address =========== 0 0x3C 1 0x3D"
- note removed: "Interface BS1 BS2 =================== SPI 0 0 I2C 1 0 8-bit (6800) 0 1 8-bit (8080) 1 1"
- note removed: "Interface selection"
- note removed: "Jim Lindblom"
- note removed: "Power Supply"
- note removed: "Short D1 (SDAin) and D2 (SDAout) in I2C mode."
- note removed: "The D/C jumper should be open if SPI or parallel interfaces are used. In those interfaces this pin determines whether incoming signals are data or command."
- note removed: "The OLED requires a 1.65-3.3V supply for its logic circuits (VDD) and a 7-7.5V supply for it's display circuitry (VCC). Fortunately, it features a charge-pump boost converter to generate a 7V supply (VCC) from 3.3-4.2V. The charge-pump input voltage is taken from the VBAT line. SJ3, closed by default, shorts the VDD and VBAT lines. This way the same supply you're using to power the logic can be b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"
- note removed: "The SSD1306 can be controlled via SPI, I2C, or a parallel interface. Use the BS1 & BS2 jumpers to select the interface. The breakout defaults to SPI (BS1 and BS2 connected to ground/0)."
- note removed: "VCC (7.0-7.5V) will be generated by on-board DC-DC converter, as long as C3 and C2 are present. It's boosted up from VBAT."
- note removed: "VCC current (Externally supplied) = 1.7-6.9mA"
- note removed: "VCC current (Internally generated) = 5.8-20.9mA"
- note removed: "VDD current < 300 uA"
- note removed: "v04"
- note removed: "v10"
- moved on the sheet: ARDUINO_NANO1, JP5, JP6

Commit message: Commit final version of PCB
Parts:
- removed C10, C8: 10uF, SparkFun-Capacitors:10UF10V10%(0805)
- removed C6: 1.0uF, SparkFun-Capacitors:1.0UF-16V-10%(0603)
- removed C7: 0.47uF, SparkFun-Capacitors:CAP0603-CAP
- removed C9: 1.0uF, SparkFun-Capacitors:1.0UF50V10%(1206)
- removed D3: BLUE, SparkFun-LED:LED-BLUE0603
- removed D4: RED, SparkFun-LED:LED-RED0603
- removed FID3, FID4: FIDUCIAL1X2, SparkFun-Aesthetics:FIDUCIAL1X2
- removed JP14: (no value), SparkFun-Connectors:USB-ABCONN-11794
- removed JP15: (no value), SparkFun-Connectors:JST_2MM_MALE
- removed JP19, JP20: (no value), SparkFun-Connectors:M023.5MM-NO_SILK
- removed JP22: (no value), SparkFun-Connectors:M02-JST-2-PTH-NO_SILK
- removed JP23, JP26: (no value), SparkFun-Connectors:M021X02_NO_SILK
- removed JP25: (no value), SparkFun-Connectors:M01PTH_NO_SILK_YES_STOP
- removed R18: 0.01, SparkFun-Resistors:RESISTOR1206
- removed R19, R20: 4.7K, SparkFun-Resistors:4.7KOHM-1/10W-1%(0603)
- removed R21: 590, SparkFun-Passives:RESISTOR0603-RES
- removed R22: 1.1k, SparkFun-Passives:RESISTOR0603-RES
- removed R23: 180, SparkFun-Resistors:180OHM1/10W1%(0603)
- removed R24: 1K, SparkFun-Resistors:1KOHM-1/10W-1%(0603)
- removed R25, R32: 100k, SparkFun-Resistors:100KOHM-1/10W-1%(0603)
- removed R26, R27, R30, R34: 10K, SparkFun-Resistors:10KOHM-1/10W-1%(0603)0603
- removed R28: ILIM, SparkFun-Resistors:RESISTORPTH-1/6W
- removed R29: ISET, SparkFun-Resistors:RESISTORPTH-1/6W
- removed R31: TMR, SparkFun-Resistors:RESISTORPTH-1/6W
- removed R33: TS, SparkFun-Resistors:RESISTORPTH-1/6W
- removed S3: (no value), SparkFun-Electromechanical:SWITCH-SPDT-SMD-A
- removed S4: (no value), SparkFun-Electromechanical:SW_DIP-2-SMT-HALFSIZE
- removed SJ10: JUMPER-PAD-3-2OF3_NC_BY_TRACE_SMALL, SparkFun-Passives:JUMPER-PAD-3-2OF3_NC_BY_TRACE_SMALL
- removed SJ6, SJ7, SJ8, SJ9: JUMPER-PAD-2-NC_BY_TRACE, SparkFun-Passives:JUMPER-PAD-2-NC_BY_TRACE
- removed TP3, TP4: TEST-POINT3X4, SparkFun-Passives:TEST-POINT3X4
- removed U3: BQ27441-G1, battery-management-temp:BQ27441-G1
- removed U4: BQ24075, battery-management-temp:BQ24075
- added J1: (no value), SparkFun-Connectors:CONN_04X2
- added S1: (no value), switch-omron:10-XX
- added U1: MAX16054AZT+, MAX16054AZT:MAX16054AZT+
Connections:
- removed net !CHG!1: R23.2, U4.!CHG!
- removed net !PGOOD!1: SJ10.1, U4.!PGOOD!
- removed net 1.8V: C7.1, JP25.1, U3.VDD
- removed net D+: JP14.D+, TP4.1
- removed net D-: JP14.D-, TP3.1
- removed net EN1: R26.2, S4.4, U4.EN1
- removed net EN2: R27.2, S4.3, U4.EN2
- removed net ILIM1: R28.2, SJ7.2, U4.ILIM
- removed net ISET1: R29.2, SJ8.2, U4.ISET
- removed net N$10: R22.1, SJ7.1
- removed net N$13: R21.1, SJ8.1
- removed net N$14: R24.2, SJ10.2
- removed net N$6: D3.C, R23.1
- removed net N$7: D4.C, R24.1
- removed net N$8: R32.2, S3.O
- removed net N$9: R30.1, SJ6.2
- removed net OUT: C8.1, D3.A, D4.A, JP20.1, JP21.2, JP22.2, R26.1, R27.1, U4.OUT
- removed net SHIELD: JP14.SHIELD
- removed net TMR1: R31.2, SJ9.2, U4.TMR
- removed net TS: R30.2, R33.2, U3.BIN, U4.TS
- removed net USB_ID: JP14.USBID
- removed net V_BATT: C10.1, R18.1, R32.1, U3.SRN, U4.BAT
- removed net V_USB: C9.1, JP14.VBUS, JP19.1, JP23.1, JP26.1, U4.IN
- new net AOFF: ARDUINO_NANO1.D7, U1.CLEAR
- new net LTB: ARDUINO_NANO1.D2, J1.2
- new net LTL: ARDUINO_NANO1.D3, J1.4
- new net LTS: ARDUINO_NANO1.D4, J1.6
- new net N$4: S1.S, U1.IN
- new net TLV+: J1.5, JP2.6
- new net TLV-: J1.7, JP2.5
- new net TSV+: J1.1, JP4.6
- new net TSV-: J1.3, JP4.5
- net !CE!: no longer R25.1, U4.!CE!
- net 3V3: now also JP21.2
- net BATTERY_IN: now also U1.VCC; no longer C6.1, JP15.+, R18.2, U3.BAT, U3.SRP
- net GND: now also J1.8, S1.P, U1.GND; no longer C10.2, C6.2, C7.2, C8.2, C9.2, JP14.GND, JP15.-, JP19.2, JP20.2, JP22.1, JP23.2, JP26.2, R21.2, R22.2, R25.2, R28.1, R29.1, R31.1, R33.1, S3.S, S4.1, S4.2, SJ10.3, SJ6.1, SJ9.1, U3.PWPD, U3.VSS, U4.EP, U4.VSS
- net GPOUT: no longer R34.1, U3.GPOUT
- net LV+: no longer JP2.6
- net LV-: no longer JP2.5
- net SCL: no longer R20.1, U3.SCL
- net SDA: no longer R19.1, U3.SDA
- net SV+: no longer JP4.6
- net SV-: no longer JP4.5
- net SYSOFF: now also U1.!OUT; no longer S3.P, U4.SYSOFF
- net V_PU: no longer R19.2, R20.2, R34.2
Other:
- note removed: "- Connect TS to 10k NTC thermistor in the battery pack. - Connect a 10k resistor to GND if TS is not used."
- note removed: "BQ24075 - 1.5A USB-Friendly LiPo Battery Charger & Power-Path Management"
- note removed: "BQ27441-G1 Fuel Gauge"
- note removed: "Battery Range: 3.3-4.2V"
- note removed: "Charge Current Select"
- note removed: "EN2 EN1 Current 0 0 100mA 0 1 500mA 1 0 ISET 1 1 Standby"
- note removed: "I2C ADDR: 0x55"
- note removed: "I2C Pull-Ups"
- note removed: "ILIM - System/Load Current Limit"
- note removed: "ISET-Charge Current"
- note removed: "OUT is the power-path management output. It manages current supplied from the USB input to both the battery and system. Or supplies battery power to the system when USB is not connected. OUT supply w/ USB: V_USB - 0.3V OUT supply w/o USB: V_BAT - 0.05V"
- note removed: "SJ1: Cut to disable TS bypass."
- note removed: "SJ2: Cut to enable charge timer."
- note removed: "SJ3: Cut to set custom ISET."
- note removed: "SJ4: Cut to set custom ILIM."
- note removed: "SJ5 sets the operation of the power LED. To either: - Power OUT indicator - !PGOOD! indicator (Good IN supply) - Open (LED disconnected)"
- note removed: "SYSOFF controls supply to the V_OUT pin. SYSOFF is active-high HIGH=OFF LOW=ON"
- note removed: "Sets combined system load and battery charge currents pulled from USB input. - I_INMAX=1650 / R_ILIM - R_ILIM range: 1.1k-8k - EX: R_ILIM = 1.1k : I_INMAX = 1.5A"
- note removed: "Sets fast charge current - R_ISET range: 590-8.9k - I_CHG = ~885 / R_ISET - EX: R_ISET = 590 : I_CHG = 1.5A"
- note removed: "Sets pre-charge and fast-charge safety timers. - Leave unconnected to set default (30min pre, 5hr charge time) - Connect to GND to disable - R_TMR range: 18k-72k - T_PRE range: 1400-2160 s - T_PRE (s) = 0.048 * R_TMR - T_MAX (s) = 10 * T_PRE"
- note removed: "Shutoff Switch"
- note removed: "Supply Input"
- note removed: "Supply range: 4.35-6.4V"
- note removed: "TMR - Saftey Timers"
- note removed: "TS - External Thermistor"
- note removed: "VDD is 1.8V generated internally"
- note removed: "V_PU is an externally supplied voltage to set the pull-up resistor HIGH voltage. Allowable range: 1.62-6V"
- moved on the sheet: ARDUINO_NANO1, JP16, JP17, JP18, JP21, JP24
